File: Electronics_Base/HW_02/hw-02-project/hw-02-prj.kicad_sch (KiCad schematic)
At the start: 2 parts, among them U1 BL0910, U2 XS2184

Commit message: add zip
Parts:
- removed U1: BL0910, hw-02-footprint-prj:My_LQFP48, symbol hw-02-lib:BL0910
- removed U2: XS2184, hw-02-footprint-prj:My_QFN48L, symbol hw-02-lib:XS2184
