File: Electronics_Base/HW_09/zelenin-HW09-prj/zelenin-HW09-prj.kicad_pcb (KiCad board)
At the start: 2 copper layers, 50.6 x 37.1 mm, 31 parts, among them J1 DC_12V, Q1 BC337, SW1 SW_Push, U1 NE555P, U2 NE555P, U3 LM317_TO-220

Commit message: update HW09
Parts:
- C12: value 2.2uF -> 1uF
- R11: value 51k -> 100k
Changed lines of the file:
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@@
 			)
 		)
-		(property "Value" "51k"
+		(property "Value" "100k"
 			(at 3.81 1.92 0)
 			(layer "F.Fab")
@@
 			)
 		)
-		(property "Value" "2.2uF"
+		(property "Value" "1uF"
 			(at -4.5 1 0)
 			(layer "F.Fab")
