File: Electronics_Base/HW_09/zelenin-HW09-prj/zelenin-HW09-prj.kicad_sch (KiCad schematic)
At the start: 31 parts, among them J1 DC_12V, Q1 BC337, SW1 SW_Push, U1 NE555P, U2 NE555P, U3 LM317_TO-220

Commit message: update HW09
Parts:
- removed C3: 0.1uF, Capacitor_THT:C_Disc_D3.0mm_W2.0mm_P2.50mm, symbol Device:C
- C12: value 2.2uF -> 1uF
- R11: value 51k -> 100k
Changed lines of the file:
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@@
-	)
-	(junction
-		(at 97.79 66.04)
-		(diameter 0)
-		(color 0 0 0 0)
 	)
 	(junction
@@
 		(color 0 0 0 0)
 	)
-	(junction
-		(at 111.76 59.69)
-		(diameter 0)
-		(color 0 0 0 0)
-	)
 	(wire
 		(pts
@@
 	(wire
 		(pts
-			(xy 97.79 66.04) (xy 101.6 66.04)
-		)
-		(stroke
-			(width 0)
-			(type default)
-		)
-	)
-	(wire
-		(pts
 			(xy 157.48 77.47) (xy 162.56 77.47)
 		)
@@
 	(wire
 		(pts
-			(xy 109.22 66.04) (xy 111.76 66.04)
-		)
-		(stroke
-			(width 0)
-			(type default)
-		)
-	)
-	(wire
-		(pts
 			(xy 93.98 105.41) (xy 91.44 105.41)
 		)
@@
 	(wire
 		(pts
-			(xy 111.76 59.69) (xy 111.76 66.04)
-		)
-		(stroke
-			(width 0)
-			(type default)
-		)
-	)
-	(wire
-		(pts
 			(xy 105.41 95.25) (xy 111.76 95.25)
 		)
@@
 	(wire
 		(pts
-			(xy 111.76 59.69) (xy 120.65 59.69)
+			(xy 110.49 59.69) (xy 120.65 59.69)
 		)
 		(stroke
@@
 		(pts
 			(xy 171.45 44.45) (xy 172.72 44.45)
-		)
-		(stroke
-			(width 0)
-			(type default)
-		)
-	)
-	(wire
-		(pts
-			(xy 110.49 59.69) (xy 111.76 59.69)
 		)
 		(stroke
@@
 			)
 		)
-		(property "Value" "51k"
+		(property "Value" "100k"
 			(at 67.056 44.45 90)
 			(effects
@@
 	(symbol
 		(lib_id "Device:C")
-		(at 105.41 66.04 90)
-		(unit 1)
-		(exclude_from_sim no)
-		(in_bom yes)
-		(on_board yes)
-		(dnp no)
-		(property "Reference" "C3"
-			(at 104.1399 62.23 90)
-			(effects
-				(font
-					(size 1.27 1.27)
-				)
-				(justify left)
-			)
-		)
-		(property "Value" "0.1uF"
-			(at 107.95 70.866 90)
-			(effects
-				(font
-					(size 1.27 1.27)
-				)
-				(justify left)
-			)
-		)
-		(property "Footprint" "Capacitor_THT:C_Disc_D3.0mm_W2.0mm_P2.50mm"
-			(at 109.22 65.0748 0)
-			(effects
-				(font
-					(size 1.27 1.27)
-				)
-				(hide yes)
-			)
-		)
-		(property "Datasheet" "~"
-			(at 105.41 66.04 0)
-			(effects
-				(font
-					(size 1.27 1.27)
-				)
-				(hide yes)
-			)
-		)
-		(property "Description" "Unpolarized capacitor"
-			(at 105.41 66.04 0)
-			(effects
-				(font
-					(size 1.27 1.27)
-				)
-				(hide yes)
-			)
-		)
-		(pin "2"
-		)
-		(pin "1"
-		)
-		(instances
-			(project "zelenin-HW09-prj"
-				(path "/02c04fff-e557-4b91-b113-92a180c13edf"
-					(reference "C3")
-					(unit 1)
-				)
-			)
-		)
-	)
-	(symbol
-		(lib_id "Device:C")
 		(at 130.81 119.38 0)
 		(unit 1)
@@
 			)
 		)
-		(property "Value" "2.2uF"
+		(property "Value" "1uF"
 			(at 68.58 71.5009 0)
 			(effects
