File: Electronics_Base/HW_10/zelenin-HW10/zelenin-HW10.kicad_sch (KiCad schematic)
At the start: 17 parts, among them J1 LOAD, J2 DC_12V, Q1 BC337, Q2 IRLZ44N, Q3 BC327, U1 NE555P

Commit message: Update HW10
Parts:
- R2: value 10k -> 5k
Changed lines of the file:
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@@
 			)
 		)
-		(property "Value" "10k"
+		(property "Value" "5k"
 			(at 145.288 59.69 90)
 			(effects
