File: Electronics_Base/HW_12/zelenin-HW12-prj/Power.kicad_sch (KiCad schematic)
At the start: 21 parts, among them J1 Vin, U4 MC34063AP, U5 LM7805_TO220

Commit message: update HW12
Parts:
- C10, C12, C9: footprint (none) -> Capacitor_THT:CP_Radial_D8.0mm_P3.80mm
- C13: footprint (none) -> Capacitor_THT:CP_Radial_D5.0mm_P2.50mm
- C14: footprint (none) -> Capacitor_THT:C_Disc_D3.0mm_W2.0mm_P2.50mm
- J1: footprint (none) -> TerminalBlock_Phoenix:TerminalBlock_Phoenix_MKDS-1,5-2-5.08_1x02_P5.08mm_Horizontal
- L1: footprint (none) -> Inductor_THT:L_Radial_D7.2mm_P3.00mm_Murata_1700
- R21, R22, R23, R24, R25, R26, R27, R28, R29, R30: footprint (none) -> Resistor_THT:R_Axial_DIN0207_L6.3mm_D2.5mm_P2.54mm_Vertical
Connections:
- net at R25.2, R26.1: now also R21.2, R24.1, R27.2, R28.1, R29.2
Other:
- moved on the sheet: R24, R26, R28
