File: Electronics_Base/HW_12/zelenin-HW12-prj/zelenin-HW12-prj.kicad_sch (KiCad schematic)
At the start: 41 parts, among them Q1 BC337, U1 74HC595, U2 74HC595

Commit message: update HW12
Parts:
- C1, C3: footprint (none) -> Capacitor_THT:CP_Radial_D8.0mm_P3.80mm
- D1, D10, D11, D12, D13, D14, D15, D16, D2, D3, D4, D5, D6, D7, D8, D9: footprint (none) -> LED_THT:LED_D5.0mm
- R1, R10, R11, R12, R13, R14, R15, R16, R17, R2, R3, R4, R5, R6, R7, R8, R9: footprint Resistor_THT:R_Axial_DIN0204_L3.6mm_D1.6mm_P7.62mm_Horizontal -> Resistor_THT:R_Axial_DIN0207_L6.3mm_D2.5mm_P2.54mm_Vertical
- R31: renamed from R?; footprint Resistor_THT:R_Axial_DIN0204_L3.6mm_D1.6mm_P7.62mm_Horizontal -> Resistor_THT:R_Axial_DIN0207_L6.3mm_D2.5mm_P2.54mm_Vertical
- U1, U2: footprint (none) -> Package_DIP:DIP-16_W7.62mm
Other:
- moved on the sheet: C1, C2
