File: Electronics_Base/CW/Zelenin-CW-power-prj/Zelenin-CW-power-prj.kicad_sch (KiCad schematic)
At the start: 47 parts, among them J1 DC_IN, J2 Conn_01x03_Pin, Q1 BC337, SW1 SW_Push, U1 MC34063AP, U2 LM7805_TO220, U3 NE555P, U4 NE555P

Commit message: Add arduino HW
Parts:
- C10: value 614p -> 610p
- R11: value 1k -> 220
Changed lines of the file:
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@@
 			)
 		)
-		(property "Value" "614p"
+		(property "Value" "610p"
 			(at 225.806 66.294 0)
 			(effects
@@
 			)
 		)
-		(property "Value" "1k"
+		(property "Value" "220"
 			(at 141.224 70.612 90)
 			(effects
