File: Electronics_Base/CW/Zelenin-CW-power-prj/Zelenin-CW-power-prj.kicad_pcb (KiCad board)
At the start: 2 copper layers, 70 x 50 mm, 47 parts, among them J1 DC_IN, J2 Conn_01x03_Pin, Q1 BC337, SW1 SW_Push, U1 MC34063AP, U2 LM7805_TO220, U3 NE555P, U4 NE555P

Commit message: Intro HW-01
Routing:
- net +5V: track 134.0 -> 127.3 mm
- net gen: track 25.6 -> 21.5 mm
Changed lines of the file:
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@@
 		(tags "CP Radial series Radial pin pitch 2.50mm  diameter 5mm Electrolytic Capacitor")
 		(property "Reference" "C6"
-			(at -0.7 3.44 0)
+			(at -2.15 1.8 0)
 			(layer "F.SilkS")
 			(effects
@@
 		(tags "C Disc series Radial pin pitch 2.50mm  diameter 3mm width 2mm Capacitor")
 		(property "Reference" "C4"
-			(at 1.4725 -4.555 -90)
+			(at 1.3725 -4.555 -90)
 			(layer "F.SilkS")
 			(effects
@@
 		(tags "CP Radial series Radial pin pitch 3.80mm  diameter 8mm Electrolytic Capacitor")
 		(property "Reference" "C2"
-			(at -3.6 -0.6 0)
+			(at -3.5 0.7 0)
 			(layer "F.SilkS")
 			(effects
@@
 	)
 	(segment
-		(start 95.8 46.50873)
-		(end 95.8 46.5)
-		(width 1)
-		(layer "F.Cu")
-		(net 3)
-	)
-	(segment
 		(start 59.25 82.25)
 		(end 61 80.5)
@@
 	)
 	(segment
-		(start 95.8 46.5)
-		(end 92.42 43.12)
-		(width 1)
-		(layer "F.Cu")
-		(net 3)
-	)
-	(segment
 		(start 91.96 61.905)
 		(end 91.96 61.11)
@@
 	)
 	(segment
-		(start 102.135 52.84373)
-		(end 95.8 46.50873)
-		(width 1)
-		(layer "F.Cu")
-		(net 3)
-	)
-	(segment
 		(start 85.675 55.357233)
 		(end 86.155 55.837233)
@@
 	)
 	(segment
-		(start 91.96 61.905)
-		(end 93.46 63.405)
-		(width 1)
-		(layer "F.Cu")
-		(net 3)
-	)
-	(segment
-		(start 92.42 43.12)
-		(end 92.42 39)
-		(width 1)
-		(layer "F.Cu")
-		(net 3)
-	)
-	(segment
 		(start 83.5 67.3)
 		(end 85.3 65.5)
@@
 	)
 	(segment
-		(start 100.095 63.405)
-		(end 102.135 61.365)
+		(start 83.1 63.3)
+		(end 83.1 48.32)
 		(width 1)
 		(layer "F.Cu")
@@
 	)
 	(segment
+		(start 85.3 65.5)
+		(end 83.1 63.3)
+		(width 1)
+		(layer "F.Cu")
+		(net 3)
+	)
+	(segment
 		(start 42.602677 82.25)
 		(end 59.25 82.25)
@@
 	)
 	(segment
-		(start 102.135 61.365)
-		(end 102.135 52.84373)
+		(start 83.1 48.32)
+		(end 92.42 39)
 		(width 1)
 		(layer "F.Cu")
@@
 	)
 	(segment
-		(start 93.46 63.405)
-		(end 100.095 63.405)
-		(width 1)
-		(layer "F.Cu")
-		(net 3)
-	)
-	(segment
 		(start 95.89 49.8)
 		(end 86.68995 49.8)
@@
 	)
 	(segment
-		(start 91.12 37.7)
-		(end 93.66 37.7)
+		(start 84.885 50.615)
+		(end 94.96 40.54)
 		(width 0.5)
 		(layer "F.Cu")
@@
 	)
 	(segment
-		(start 91.12 44.38)
-		(end 91.12 37.7)
+		(start 94.96 40.54)
+		(end 94.96 39)
 		(width 0.5)
 		(layer "F.Cu")
@@
 	)
 	(segment
-		(start 84.885 50.615)
-		(end 91.12 44.38)
-		(width 0.5)
-		(layer "F.Cu")
-		(net 26)
-	)
-	(segment
-		(start 93.66 37.7)
-		(end 94.96 39)
-		(width 0.5)
-		(layer "F.Cu")
-		(net 26)
-	)
-	(segment
 		(start 68.68 78.82)
 		(end 73.32 78.82)
@@
 		(polygon
 			(pts
-				(xy 53.05 53.56) (xy 58.85 53.56) (xy 59.95 54.16) (xy 77.55 54.16) (xy 82.5 56.16) (xy 82.5 59.5)
-				(xy 82.5 62.5) (xy 82.5 74.5) (xy 73 74.5) (xy 70 81.4) (xy 49.3 81.3) (xy 49.3 64.8) (xy 74.9 64.8)
+				(xy 53.05 53.56) (xy 58.85 53.56) (xy 59.95 54.16) (xy 80.3 54.2) (xy 82.1 56.4) (xy 82.1 63.9)
+				(xy 82.519 64.46) (xy 82.5 74.5) (xy 73 74.5) (xy 70 81.4) (xy 49.3 81.3) (xy 49.3 64.8) (xy 74.9 64.8)
 				(xy 74.9 56.8) (xy 68.35 56.1) (xy 53.05 56.1)
 			)
